File: selektywne/sel.sch (EAGLE design)
At the start: 16 parts, among them IC2 SP3485EN-L_TR, J1 5-1634556-0, U1 ADS1248IPW, U2 TLC274CD, U3 TLC274CD, X1 RJ45-6L-B

Commit message: bck
Parts:
- added AM1G-1205D-NZ: AM1G-1205D-NZ, AM!G-NZ:AM1G-1205D-NZ
- added C10, C11, C8: 100nF, rcl:C-EUC1206
- added C4, C5: 2.2uF, rcl:C-EUC1206
- added C6, C7: 47nF, rcl:C-EUC1206
- added OK1: PC817, optocoupler:PC817
- added R10, R5: 1k, rcl:R-EU_R1206
- added R11, R8: 10k, rcl:R-EU_R1206
- added R12: 160k, rcl:R-EU_R1206
- added R6: 1.5k, rcl:R-EU_R1206
- added R7: 4.7k, rcl:R-EU_R1206
- added R9: 15k, rcl:R-EU_R1206
- added U4: TPS72301DBVT, TPS72301DBVT:TPS72301DBVT
- R2: value (none) -> 4.7k
Connections:
- removed net CLS_SPI: U1.CLK
- new net -3V: C4.1, R8.2, U4.OUT
- new net -5V: AM1G-1205D-NZ.-V_O, C5.1, R7.1, U4.IN
- new net DRDY_MC: ESP32_H_2.13, OK1.COL, R11.2
- new net FB: R8.1, R9.2, U4.FB
- new net N$5: AM1G-1205D-NZ.CNTL, R5.2, R6.2
- new net N$6: R7.2, U4.EN
- new net N$7: OK1.A, R10.1
- new net N$8: C8.2, U1.VREFOUT
- new net N$9: R12.1, U1.START
- net +12V: now also AM1G-1205D-NZ.V_IN, R5.1
- net +3V3: now also AT1.VDD1, AT1.VDD2, C10.2, C11.2, C6.2, C7.2, R11.1, R12.2
- net +5V: now also AM1G-1205D-NZ.+V_O
- net CLK_SPI: now also U1.SCLK
- net DRDY: now also R10.2
- net GND: now also AM1G-1205D-NZ.GND, AT1.GND1_1, AT1.GND1_2, AT1.GND2_1, AT1.GND2_2, C10.1, C11.1, C4.2, C5.2, C6.1, C7.1, C8.1, OK1.C, OK1.EMIT, R6.1, R9.1, U1.CLK, U1.VREFCOM, U4.GND
Other:
- moved on the sheet: AT1, C1, C2, C3, J1, R1, R3, R4, U1, U2, U3

Commit message: fixed power supply
Parts:
- removed R12: 160k, rcl:R-EU_R1206
- added C9: 100nF, rcl:C-EUC1206
- added OK2: PC817, optocoupler:PC817
- added R13: 1k, rcl:R-EU_R1206
- added R14: 10k, rcl:R-EU_R1206
- added R15: 4.7k, rcl:R-EU_R1206
Connections:
- removed net -3V: C4.1, R8.2, U4.OUT
- removed net CS: AT1.OUT1, U1.!CS
- removed net D5_CS: AT1.IN1, ESP32_H_2.8
- removed net N$9: R12.1, U1.START
- new net +2_5V: C11.2, U1.AVDD
- new net -2_5V: C4.1, C9.1, R8.2, U1.AVSS, U4.OUT
- new net N$10: OK2.A, R13.1
- new net N$11: R15.1, U1.!CS
- new net RESET: AT1.IN1, ESP32_H_2.11, ESP32_H_2.8
- new net START: OK2.COL, R14.2, U1.START
- new net START_MC: ESP32_H_2.4, R13.2
- net +3V3: now also R14.1; no longer C11.2, R12.2, U1.AVDD
- net +5V: now also U2.VDD, U3.VDD
- net -5V: now also U2.GND, U3.GND
- net DRDY_MC: now also ESP32_H_2.14; no longer ESP32_H_2.13
- net GND: now also C9.2, OK2.C, OK2.EMIT, R15.2; no longer U1.AVSS
- net RESET_ADC: now also AT1.OUT1
Other:
- note added: "???????????: -ESP32, EN pin pull up -Eth piny kom. -Zasilanie ogólnie -Piny do ADC RST, START, CS DRDY -Zasilanie HCPL -Przetwornica na esp czy może 3v3 -napiecie z tps -2.5v ? do adc -jak maja byc zasilane wzmacniacze =/- 2.5v ? -ADC: start na high t od zasilenia do start na 1, RESET -Analogi, anty-aliansing filtr 20kbs 300mOhm"
- note added: "ADC"
- note added: "D34"
- note added: "ESP32_devboar"
- note added: "Kanały analogowe"
- note added: "Komunikacja"
- note added: "Zasilanie"
- moved on the sheet: AT1, C10, C11, C6, C7, C8, OK1, R10, R11, U1

Commit message: fixed some errors
Parts:
- removed OK2: PC817, optocoupler:PC817
- removed R13, R5: 1k, rcl:R-EU_R1206
- removed R14: 10k, rcl:R-EU_R1206
- removed R6: 1.5k, rcl:R-EU_R1206
- removed X1: RJ45-6L-B, con-tycoelectronics:RJ45-6L-B
- added C12: 10uF, rcl:C-EUC1206
- added C13, C14, C15, C16: 100nF, rcl:C-EUC1206
- added C17: 1uF, rcl:C-EUC1206
- added IC1: TPS70925DBVT, SamacSys_Parts:TPS70925DBVT
- added X2: 0446200002, con-molex:0446200002
- R2: value 4.7k -> 1k
Connections:
- net -2_5V renamed -2_5V_OP
- removed net +2_5V: C11.2, U1.AVDD
- removed net N$10: OK2.A, R13.1
- removed net N$5: AM1G-1205D-NZ.CNTL, R5.2, R6.2
- new net +2_5V_OP: C11.2, IC1.OUT, U1.AVDD
- new net +5V_OP: AM1G-1205D-NZ.+V_O, AT1.VDD2, C10.2, C14.1, C7.2, IC1.IN, R2.2, U1.DVDD
- new net -5V_OP: AM1G-1205D-NZ.-V_O, C5.1, R7.1, U4.IN
- new net GND_OP: AM1G-1205D-NZ.COMM, AT1.GND2_1, AT1.GND2_2, C10.1, C11.1, C14.2, C17.2, C4.2, C5.2, C7.1, C8.1, C9.2, IC1.GND, R15.2, R9.1, U1.CLK, U1.DGND, U1.VREFCOM, U4.GND
- net +12V: now also C12.2, C13.2, X2.1; no longer R5.1, X1.1
- net +3V3: now also C15.2; no longer AT1.VDD2, C10.2, C7.2, R14.1, R2.2, U1.DVDD
- net +5V: now also C16.1, X2.2; no longer AM1G-1205D-NZ.+V_O
- net -5V: no longer AM1G-1205D-NZ.-V_O, C5.1, R7.1, U4.IN
- net EN: no longer R2.1
- net GND: now also C12.1, C13.1, C15.1, C16.2, X2.8; no longer AT1.GND2_1, AT1.GND2_2, C10.1, C11.1, C4.2, C5.2, C7.1, C8.1, C9.2, OK2.C, OK2.EMIT, R15.2, R6.1, R9.1, U1.CLK, U1.DGND, U1.VREFCOM, U4.GND, X1.8
- net N$1: now also X2.4; no longer X1.4
- net N$2: now also X2.3; no longer X1.5
- net N$3: no longer J1.1
- net START: now also C17.1, R2.1; no longer OK2.COL, R14.2
- net START_MC: no longer R13.2
Other:
- note added: "Opoźnienie ok. 2ms"
- note added: "Poprawic dzielnik na 2.5"
- note added: "Sprawdzic co z tym controlem"
- note removed: "???????????: -ESP32, EN pin pull up -Eth piny kom. -Zasilanie ogólnie -Piny do ADC RST, START, CS DRDY -Zasilanie HCPL -Przetwornica na esp czy może 3v3 -napiecie z tps -2.5v ? do adc -jak maja byc zasilane wzmacniacze =/- 2.5v ? -ADC: start na high t od zasilenia do start na 1, RESET -Analogi, anty-aliansing filtr 20kbs 300mOhm"
- note removed: "ADC"
- moved on the sheet: AT1, C10, C11, C4, C5, C6, C7, C8, C9, OK1, R10, R11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

Commit message: Fixed analog and digital problems,a active filter
Parts:
- removed C3: 100nF, rcl:C-EUC1206
- removed OK1: PC817, optocoupler:PC817
- added C21, C22, C23, C24, C25, C26, C27, C33, C34, C35, C36: 2.2uF, rcl:C-EUC1206
- added C28, C29, C30, C31, C32: 100nF, rcl:C-EUC1206
- added J2, J3, J4, J5, J6, J7, J8: 5-1634556-0, 5-1634556-0:5-1634556-0
- added R12, R36, R37, R38, R39: 160k, rcl:R-EU_R1206
- added R16, R17, R18, R19, R20, R21, R22, R28, R29, R30, R31: 6.8k, rcl:R-EU_R1206
- added R23, R24, R25, R26, R27: 1k, rcl:R-EU_R1206
- added R5, R6: 47, rcl:R-EU_R1206
- added U5, U6: TLC274CD, TLC274CD:TLC274CD
- C2: value 100nF -> 2.2uF
- R10: value 1k -> 47
- R11: value 10k -> 47
- R3: value 160k -> 6.8k
- R8: value 10k -> 51k
- R9: value 15k -> 47k
Connections:
- net D18_CLK renamed MC_SCLK
- net D19_MISO renamed MC_MISO/!DRDY
- net D23_MOSI renamed MC_MOSI
- net D4_RST renamed DIR
- removed net -5V: U2.GND, U3.GND
- removed net DRDY: R10.2, U1.!DRDY
- removed net DRDY_MC: ESP32_H_2.14, OK1.COL, R11.2
- removed net MISO: AT1.IN4, U1.DOUT/~DRDY
- removed net RESET: AT1.IN1, ESP32_H_2.11, ESP32_H_2.8
- removed net START_MC: ESP32_H_2.4
- new net IRQ_!DRDY: ESP32_H_2.11
- new net MC_RESET: AT1.IN1, ESP32_H_2.8
- new net MISO/!DRDY: AT1.IN4, R11.2, U1.DOUT/~DRDY
- new net N$10: R11.1
- new net N$12: R12.1, U3.2IN-
- new net N$13: U6.1IN+
- new net N$15: U3.2IN+
- new net N$18: R16.1, U2.1IN+
- new net N$19: C2.1, C21.1, R16.2, R3.1
- new net N$20: R18.1, U2.2IN+
- new net N$21: C22.1, C23.1, R17.1, R18.2
- new net N$22: R20.1, U2.3IN+
- new net N$23: C24.1, C25.1, R19.1, R20.2
- new net N$24: R22.1, U2.4IN+
- new net N$25: C26.1, C27.1, R21.1, R22.2
- new net N$31: R29.1, U5.1IN+
- new net N$32: C33.1, C34.1, R28.1, R29.2
- new net N$33: R31.1, U5.2IN+
- new net N$34: C35.1, C36.1, R30.1, R31.2
- new net N$35: U5.3IN+
- new net N$37: U5.4IN+
- new net N$44: R36.1, U6.1IN-
- new net N$45: R37.1, U6.2IN-
- new net N$46: R38.1, U6.3IN-
- new net N$47: R39.1, U6.4IN-
- new net N$48: U6.2IN+
- new net N$49: U6.3IN+
- new net N$5: R5.1
- new net N$50: U6.4IN+
- new net N$9: R10.1
- new net OUT2: C23.2, R24.2, U2.2IN-, U2.2OUT
- new net OUT2_WT: R17.2, R37.2, U6.2OUT
- new net OUT3: C25.2, R25.2, U2.3IN-, U2.3OUT
- new net OUT3_WT: R19.2, R38.2, U6.3OUT
- new net OUT4: C27.2, R1.2, U2.4IN-, U2.4OUT
- new net OUT4_WT: R21.2, R39.2, U6.4OUT
- new net OUT5: C34.2, R26.2, U5.1IN-, U5.1OUT
- new net OUT5_WT: R28.2, R4.2, U3.1OUT
- new net OUT6: C36.2, R27.2, U5.2IN-, U5.2OUT
- new net OUT6_WT: R12.2, R30.2, U3.2OUT
- net +3V3: no longer R11.1
- net +5V: no longer U2.VDD, U3.VDD
- net +5V_OP: now also U2.VDD, U3.VDD, U5.VDD, U6.VDD
- net -5V_OP: now also U2.GND, U3.GND, U5.GND, U6.GND
- net CH0: now also C28.1, R23.1; no longer C1.1, R1.1
- net CH1: now also C29.1, R24.1
- net CH2: now also C30.1, R25.1
- net CH4: now also C1.1, R1.1
- net CH5: now also C31.1, R26.1
- net CH6: now also C32.1, R27.1
- net CLK_SPI: now also R6.2
- net GND: no longer C1.2, C2.2, C3.2, J1.2, OK1.C, OK1.EMIT
- net GND_OP: now also C1.2, C2.2, C22.2, C24.2, C26.2, C28.2, C29.2, C30.2, C31.2, C32.2, C33.2, C35.2, J1.2, J2.2, J3.2, J4.2, J5.2, J6.2, J7.2, J8.2
- net MOSI: now also R10.2
- net N$3: no longer C3.1
- net N$7: now also R6.1; no longer OK1.A, R10.1
- net OUT1: now also C21.2, R23.2, U2.1IN-; no longer C2.1, R1.2, R3.1, U2.1IN+
- net OUT1_WT: now also R36.2, U6.1OUT; no longer R4.2, U3.1OUT
- net RESET_ADC: now also R5.2
Other:
- note added: "Filtry AA"
- note added: "Filtry z kondesatora styrofleksowego"
- note added: "Low pass active filter Fcut = 11 Hz"
- note added: "RC"
- note added: "Vout = -1.186(1+R8/R9) R8+R9 = 100k"
- note added: "Wejścia BNC"
- note added: "Wtórnik"
- note removed: "Anty-aliansing filtr"
- note removed: "ESP32_devboar"
- note removed: "Kanały analogowe"
- note removed: "Komunikacja"
- note removed: "Low pass filtr Fcut = 10Hz"
- note removed: "Poprawic dzielnik na 2.5"
- note removed: "Wtornik napięcia"
- note removed: "Zasilanie"
- note removed: "kondensator ten na s xd"
- moved on the sheet: AM1G-1205D-NZ, AT1, C1, C10, C11, C13, C14, C17, C2, C4, C5, C6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

Commit message: fixes in progress 8/12
Parts:
- added C18: 10uF, rcl:C-EUC1206
- added C19, C20, C38, C39, C40, C41, C42, C43, C44, C46, C48, C50, C52, C54, C56, C58, C60: 2.2uF, rcl:C-EUC1206
- added C3, C37, C45, C47, C49, C51, C53, C55, C57, C59: 100nF, rcl:C-EUC1206
- added L1, L2: (no value), rcl:L-US0204/7
- added R13, R14, R32, R33, R34, R35: 10k, rcl:R-EU_R1206
- C13, C16: value 100nF -> 2.2uF
- C6, C7: value 47nF -> 100nF
- R1, R23, R24, R25, R26, R27: value 1k -> 10k
Connections:
- removed net +2_5V_OP: C11.2, IC1.OUT, U1.AVDD
- removed net +5V_OP: AM1G-1205D-NZ.+V_O, AT1.VDD2, C10.2, C14.1, C7.2, IC1.IN, R2.2, U1.DVDD, U2.VDD, U3.VDD, U5.VDD, U6.VDD
- removed net N$35: U5.3IN+
- removed net N$37: U5.4IN+
- new net 2_5V_OP: C11.2, C43.2, IC1.OUT, U1.AVDD
- new net 5V_OP: AM1G-1205D-NZ.+V_O, AT1.VDD2, C10.2, C14.1, C39.1, C41.1, C42.2, C45.1, C46.1, C47.1, C48.1, C49.1, C50.1, C51.1, C52.1, C7.1, IC1.IN, R2.2, U1.DVDD, U2.VDD, U3.VDD, U5.VDD, U6.VDD
- new net N$16: C52.2
- net +12V: now also C12.1, C20.1, C37.2, L2.2; no longer C12.2
- net +3V3: now also C19.2, C40.2
- net +5V: now also C18.1, C3.1, L1.1
- net -2_5V_OP: now also C44.1
- net -5V_OP: now also C38.1, C53.2, C54.2, C55.2, C56.2, C57.2, C58.2, C59.2, C60.2
- net CH0: now also R13.2
- net CH1: now also C1.1, R1.1, R14.2; no longer C29.1, R24.1
- net CH2: now also C29.1, R24.1, R25.2; no longer C30.1, R25.1
- net CH3: now also C30.1, R26.1, R27.2
- net CH4: now also C31.1, R32.1, R33.2; no longer C1.1, R1.1
- net CH5: now also C32.1, R34.1, R35.2; no longer C31.1, R26.1
- net CH6: no longer C32.1, R27.1
- net GND: now also C12.2, C18.2, C19.1, C20.2, C3.2, C37.1, C40.1, L1.2, L2.1; no longer C12.1
- net GND_OP: now also C38.2, C39.2, C41.2, C42.1, C43.1, C44.2, C45.2, C46.2, C47.2, C48.2, C49.2, C50.2, C51.2, C53.1, C54.1, C55.1, C56.1, C57.1, C58.1, C59.1, C60.1, C7.2, R13.1, R14.1, R25.1, R27.1, R33.1, R35.1; no longer C7.1
- net OUT2: now also R1.2; no longer R24.2
- net OUT3: now also R24.2; no longer R25.2
- net OUT4: now also R26.2; no longer R1.2
- net OUT5: now also R32.2; no longer R26.2
- net OUT6: now also R34.2; no longer R27.2
Other:
- note added: "Do resetu ESP32 z poziomu programu"
- note added: "Filtry AA + dzielniki"
- note removed: "Filtry AA"

Commit message: fixes 12/12
Parts:
- removed C35, C36, C48, C50, C58, C60: 2.2uF, rcl:C-EUC1206
- removed C47, C49, C57, C59: 100nF, rcl:C-EUC1206
- removed J5: 5-1634556-0, 5-1634556-0:5-1634556-0
- removed R21, R22, R28, R29, R30, R31: 6.8k, rcl:R-EU_R1206
- removed U2, U5: TLC274CD, TLC274CD:TLC274CD
- added C61: 1nF, rcl:C-EUC1206
- added C62, C64, C66, C67, C68, C69: 100nF, rcl:C-EUC1206
- added C63, C65: 2.2uF, rcl:C-EUC1206
- added JP1, JP2, JP3, JP4, JP5, JP6: (no value), pinhead:PINHD-1X1
- added L3: (no value), rcl:L-US0204/7
- added R40, R41, R42, R43, R44, R45: 160k, rcl:R-EU_R1206
- added U7: TLC274CN, TLC274CN:TLC274CN
- C2, C21, C22, C23, C24, C25, C26, C27: value 2.2uF -> 100nF
- C33: value 2.2uF -> 10uF
- R16, R17, R18, R19, R20, R3: value 6.8k -> 160k
- U3, U6: value TLC274CD -> TLC274CN; device TLC274CD:TLC274CD -> TLC274CN:TLC274CN
Connections:
- net N$1 renamed B
- net N$2 renamed A
- removed net N$22: R20.1, U2.3IN+
- removed net N$23: C24.1, C25.1, R19.1, R20.2
- removed net N$24: R22.1, U2.4IN+
- removed net N$25: C26.1, C27.1, R21.1, R22.2
- removed net N$31: R29.1, U5.1IN+
- removed net N$32: C33.1, C34.1, R28.1, R29.2
- removed net N$33: R31.1, U5.2IN+
- removed net N$34: C35.1, C36.1, R30.1, R31.2
- removed net N$49: U6.3IN+
- removed net N$50: U6.4IN+
- new net -5V_OP1: C45.2, C46.2, C51.2, C52.2, C62.2, C63.2, U3.VDD, U6.VDD, U7.VDD
- new net N$13: U7.1IN+
- new net N$14: U7.2IN+
- new net N$17: U7.3IN+
- new net N$26: U7.4IN+
- new net N$27: R41.1, U6.2IN-
- new net N$28: R42.1, U6.1IN-
- new net N$30: C68.1, C69.1, R44.1, R45.2
- new net N$37: R43.1, U3.4IN+
- new net N$38: R45.1, U3.3IN+
- net +5V: now also C33.2, C34.2, L3.1
- net -5V_OP: now also C64.2, C65.2, U7.GND; no longer C57.2, C58.2, C59.2, C60.2, U2.GND, U5.GND
- net 5V_OP: no longer C45.1, C46.1, C47.1, C48.1, C49.1, C50.1, C51.1, C52.1, U2.VDD, U3.VDD, U5.VDD, U6.VDD
- net GND: now also C33.1, C34.1, C61.2, L3.2
- net GND_OP: now also C45.1, C46.1, C51.1, C52.1, C61.1, C62.1, C63.1, C64.1, C65.1, C66.2, C68.2, J6.1, JP1.1, JP2.1, JP3.1, JP4.1, JP5.1, JP6.1; no longer C33.2, C35.2, C45.2, C46.2, C47.2, C48.2, C49.2, C50.2, C51.2, C57.1, C58.1, C59.1, C60.1, J5.2
- net N$12: now also C24.1, C25.1, R12.2, R4.1; no longer R12.1, U3.2IN-
- net N$15: now also R12.1, U3.1IN+; no longer U3.2IN+
- net N$16: now also C26.1, C27.1, R19.1, R20.2; no longer C52.2
- net N$18: now also R20.1, U3.2IN+; no longer R16.1, U2.1IN+
- net N$20: now also C66.1, C67.1, R40.1, R43.2; no longer R18.1, U2.2IN+
- net N$3: now also R18.1, U6.3IN+; no longer U3.1IN+
- net N$4: now also R16.1, U6.4IN+; no longer R4.1, U3.1IN-
- net N$44: now also U7.4IN-; no longer U6.1IN-
- net N$45: now also U7.3IN-; no longer U6.2IN-
- net N$46: now also U7.2IN-; no longer U6.3IN-
- net N$47: now also U7.1IN-; no longer U6.4IN-
- net OUT1: now also C23.2, U6.3IN-, U6.3OUT; no longer C21.2, U2.1IN-, U2.1OUT
- net OUT1_WT: now also R17.2, R39.2, U7.1OUT; no longer R3.2, R36.2, U6.1OUT
- net OUT2: now also C21.2, U6.4IN-, U6.4OUT; no longer C23.2, U2.2IN-, U2.2OUT
- net OUT2_WT: now also R3.2, R38.2, U7.2OUT; no longer R17.2, R37.2, U6.2OUT
- net OUT3: now also U3.1IN-, U3.1OUT; no longer U2.3IN-, U2.3OUT
- net OUT3_WT: now also R37.2, R4.2, U7.3OUT; no longer R19.2, R38.2, U6.3OUT
- net OUT4: now also U3.2IN-, U3.2OUT; no longer U2.4IN-, U2.4OUT
- net OUT4_WT: now also R19.2, R36.2, U7.4OUT; no longer R21.2, R39.2, U6.4OUT
- net OUT5: now also C69.2, U3.3IN-, U3.3OUT; no longer C34.2, U5.1IN-, U5.1OUT
- net OUT5_WT: now also R42.2, R44.2, U6.1OUT; no longer R28.2, R4.2, U3.1OUT
- net OUT6: now also C67.2, U3.4IN-, U3.4OUT; no longer C36.2, U5.2IN-, U5.2OUT
- net OUT6_WT: now also R40.2, R41.2, U6.2OUT; no longer R12.2, R30.2, U3.2OUT
Other:
- note added: "Dioda referencyjna"
- note added: "ESD protection ~3KV"
- note added: "IN_WT"
- note added: "Kon. styfleksowy"
- note added: "Rezystor"
- note removed: "Filtry z kondesatora styrofleksowego"
- note removed: "Low pass active filter Fcut = 11 Hz"
- note removed: "RC"
- note removed: "Wtórnik"
- moved on the sheet: C1, C12, C15, C16, C18, C19, C2, C20, C21, C22, C23, C24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

Commit message: PCB v1
Parts:
- C38: value 2.2uF -> 100uF
- L1, L2, L3: value (none) -> 30uH
Connections:
- net N$13 renamed 1IN+
- net N$14 renamed 2IN+
- net N$17 renamed 3IN+
- net N$26 renamed 4IN+
- net N$35 renamed 1IN+_2
- net N$36 renamed 2IN+_2
- net N$4 renamed 4IN+_2
- removed net -5V_OP1: C45.2, C46.2, C51.2, C52.2, C62.2, C63.2, U3.VDD, U6.VDD, U7.VDD
- net 5V_OP: now also C45.2, C46.2, C51.2, C52.2, C62.2, C63.2, U3.VDD, U6.VDD, U7.VDD
- net OUT1: now also C69.2, U3.3IN-, U3.3OUT; no longer C23.2, U6.3IN-, U6.3OUT
- net OUT1_WT: now also R44.2; no longer R17.2
- net OUT2: now also C67.2, U3.4IN-, U3.4OUT; no longer C21.2, U6.4IN-, U6.4OUT
- net OUT2_WT: now also R40.2; no longer R3.2
- net OUT5: now also C23.2, U6.3IN-, U6.3OUT; no longer C69.2, U3.3IN-, U3.3OUT
- net OUT5_WT: now also R17.2; no longer R44.2
- net OUT6: now also C21.2, U6.4IN-, U6.4OUT; no longer C67.2, U3.4IN-, U3.4OUT
- net OUT6_WT: now also R3.2; no longer R40.2
Other:
- note removed: "Sprawdzic co z tym controlem"
- note removed: "USB"

Commit message: fux wt problem
Connections:
- net 1IN+_2 renamed WT5
- removed net 2IN+_2: U6.2IN+
- removed net 4IN+_2: R16.1, U6.4IN+
- removed net N$27: R41.1, U6.2IN-
- new net 3IN+_2: R16.1, U6.3IN+
- new net N$1: R41.1, U6.4IN-
- new net WT6: U6.4IN+
- net N$3: now also U6.2IN+; no longer U6.3IN+
- net OUT5: now also U6.2IN-, U6.2OUT; no longer U6.3IN-, U6.3OUT
- net OUT6: now also U6.3IN-, U6.3OUT; no longer U6.4IN-, U6.4OUT
- net OUT6_WT: now also U6.4OUT; no longer U6.2OUT
Other:
- moved on the sheet: C2, C21, C22, C23, R16, R17, R18, R3, R41
